Commit message: 大改，增加碰撞模型，重新生成moveit_config包

File: dofbot_description/urdf/dofbot.urdf (robot description, URDF)
Before this commit: robot dofbot, 6 links, 5 joints
Links:
- added link left_finger, mass 0.006329; collision mesh filename=package://dofbot_description/meshes/collision/left_finger_c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; collision mesh filename=package://dofbot_description/meshes/collision/left_finger_c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
- added link right_finger, mass 0.005998; collision mesh filename=package://dofbot_description/meshes/collision/right_finger_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; collision mesh filename=package://dofbot_description/meshes/collision/right_finger_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
- link base_link: geometry collision mesh filename=package://dofbot_description/meshes/collision/base_link_col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; collision mesh filename=package://dofbot_description/meshes/collision/base_link_col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
- link link1: geometry collision mesh filename=package://dofbot_description/meshes/collision/link1_col.stl; visual mesh filename=package://dofbot_description/meshes/visual/link1.STL
- link link2: geometry collision mesh filename=package://dofbot_description/meshes/collision/link2_col.stl; visual mesh filename=package://dofbot_description/meshes/visual/link2.STL
- link link3: geometry collision mesh filename=package://dofbot_description/meshes/collision/link3_col.stl; visual mesh filename=package://dofbot_description/meshes/visual/link3.STL
- link link4: geometry collision mesh filename=package://dofbot_description/meshes/collision/link4_col_1.s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; collision mesh filename=package://dofbot_description/meshes/collision/link4_col_2.s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
- link link5: mass 0.139894 -> 0.091378; geometry collision mesh filename=package://dofbot_description/meshes/collision/flange_col_1.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; collision mesh filename=package://dofbot_description/meshes/collision/flange_col_2.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
Joints:
- added joint left_finger_joint: type prismatic, parent link5, child left_finger, origin xyz=0 0 0 rpy=0 0 0, axis 1 0 0, limit lower=-0.03 upper=0.03 effort=5.0 velocity=0.5
- added joint right_finger_joint: type prismatic, parent link5, child right_finger, origin xyz=0 0 0 rpy=0 0 0, axis 1 0 0, limit lower=-0.03 upper=0.03 effort=5.0 velocity=0.5, mimic joint=left_finger_joint multiplier=-1.0 offset=0.0
- joint joint1: limit lower=-1.5708 upper=1.5708 effort=1.5 velocity=1 -> lower=-1.5708 upper=1.5708 effort=1.5 velocity=3.14
- joint joint2: limit lower=-1.5708 upper=1.5708 effort=1.5 velocity=1 -> lower=-1.5708 upper=1.5708 effort=1.5 velocity=3.14
- joint joint3: limit lower=-1.5708 upper=1.5708 effort=1.5 velocity=1 -> lower=-1.5708 upper=1.5708 effort=1.5 velocity=3.14
- joint joint4: limit lower=-1.5708 upper=1.5708 effort=1.5 velocity=1 -> lower=-1.5708 upper=1.5708 effort=1.5 velocity=3.14
- joint joint5: limit lower=-1.5708 upper=3.1416 effort=0.6 velocity=1 -> lower=-1.5708 upper=3.1416 effort=0.6 velocity=3.14
