Commit message: feat: 重构机械臂描述包，新增控制与仿真接口，完善碰撞与可视化模型
- 碰撞模型优化：将link2/3/4的单一碰撞STL拆分为多段，提升碰撞检测精度
- 可视化模型更新：visual目录下的.STL统一改为小写.stl，适配文件系统
- 新增 dofbot_control 包：含硬件接口与Gazebo仿真接口(ros_control)
- 新增 dofbot_mujoco 包：MuJoCo仿真节点与启动文件
- 新增文档与工具：README、硬件手册、舵机协议、URDF尺寸参考图
- 新增 dofbot.xacro：支持参数化URDF生成
- 新增 dofbot_mjcf.xml：MuJoCo格式的机器人模型描述
- IK求解器重构：更新中英文注释与算法文档，优化代码结构
- MoveIt配置刷新：联合名称统一、关节限位更新、启动文件规范化
- package.xml统一升级为format 3，许可证改为Apache-2.0，清理冗余依赖
- CMakeLists.txt精简，移除自动生成模板中的冗余注释
- 删除 dofbot_moveit_config_backup 备份目录

Co-Authored-By: Claude Opus 4.7 <noreply@anthropic.com>

File: dofbot_description/urdf/dofbot.urdf (robot description, URDF)
Before this commit: robot dofbot, 8 links, 7 joints
Links:
- link link2: geometry collision mesh filename=package://dofbot_description/meshes/collision/link2_col_1.s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; collision mesh filename=package://dofbot_description/meshes/collision/link2_col_2.s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
- link link3: geometry collision mesh filename=package://dofbot_description/meshes/collision/link3_col_1.s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; collision mesh filename=package://dofbot_description/meshes/collision/link3_col_2.s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
- link link4: geometry collision mesh filename=package://dofbot_description/meshes/collision/link4_col_1.s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; collision mesh filename=package://dofbot_description/meshes/collision/link4_col_2.s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
