Commit message: fix: 将 gripper_tcp_joint 从 mimic 改为 fixed joint，遵循 ROS 社区标准

File: dofbot_description/urdf/dofbot.xacro (robot description, xacro)
@@ -254,12 +254,9 @@
     </collision>
   </link>
-  <!-- gripper_tcp: 夹爪末端中心虚位点, mimic 跟随 gripper_left_joint -->
-  <joint name="gripper_tcp_joint" type="prismatic">
+  <!-- gripper_tcp: 末端工具中心点 (TCP)，固定偏移，供 MoveIt IK 计算 -->
+  <joint name="gripper_tcp_joint" type="fixed">
     <origin xyz="0 0 0.0925" rpy="0 0 0"/>
     <parent link="wrist_roll_link"/>
     <child link="gripper_tcp"/>
-    <axis xyz="0 0 1"/>
-    <mimic joint="gripper_left_joint" multiplier="-0.583" offset="0"/>
-    <limit lower="-0.05" upper="0.20" effort="0" velocity="1"/>
   </joint>
   <link name="gripper_tcp">

Commit message: fix: MJCF 执行器力矩与 URDF wrist_roll effort 匹配真机舵机参数

File: dofbot_description/urdf/dofbot.xacro (robot description, xacro)
@@ -165,5 +165,5 @@
     <child link="wrist_roll_link" />
     <axis xyz="0 0 1" />
-    <limit lower="-1.5708" upper="3.1416" effort="0.6" velocity="3.14" />
+    <limit lower="-1.5708" upper="3.1416" effort="1.5" velocity="3.14" />
     <dynamics damping="0.1" friction="0.05" />
   </joint>
