Commit message: 真机调试：HardwareInterface 完备修正 + 夹爪校准 + 标准 ROS 数据管道
硬件驱动:
- 3 个旋转关节方向反转修正 (direction=-1)
- 6 路中位偏差硬校准 (mid_deviation)
- 夹爪三点实测分段映射, 物理安全边界钳位
- I2C 读操作寄存器指针偏移修复
- write 每周期执行 (消除运动卡顿)
- 堵转保护 (误差 >0.12rad × 400ms → 自动关扭矩)
- 启动防跳 (首次 write 用实际位置)

夹爪 TCP:
- 新增 gripper_tcp link + URDF mimic 自动跟随

标准化管道:
- /joint_states 为 8 关节单源标准输出 (/joint_states_raw 内部分离)
- PC 端零适配, 直读标准 topic

MoveIt:
- end_effector parent_link → gripper_tcp
- 碰撞矩阵 + RViz 着色
- 控制器管理器硬编码修正
- demo.launch 支持 fake_execution 参数

Co-Authored-By: Claude Opus 4.7 <noreply@anthropic.com>

File: dofbot_description/urdf/dofbot.xacro (robot description, xacro)
@@ -254,4 +254,20 @@
     </collision>
   </link>
+  <!-- gripper_tcp: 夹爪末端中心虚位点, mimic 跟随 gripper_left_joint -->
+  <joint name="gripper_tcp_joint" type="prismatic">
+    <origin xyz="0 0 0.0925" rpy="0 0 0"/>
+    <parent link="wrist_roll_link"/>
+    <child link="gripper_tcp"/>
+    <axis xyz="0 0 1"/>
+    <mimic joint="gripper_left_joint" multiplier="-0.583" offset="0"/>
+    <limit lower="-0.05" upper="0.20" effort="0" velocity="1"/>
+  </joint>
+  <link name="gripper_tcp">
+    <inertial>
+      <mass value="1e-9"/>
+      <origin xyz="0 0 0"/>
+      <inertia ixx="1e-15" ixy="0" ixz="0" iyy="1e-15" iyz="0" izz="1e-15"/>
+    </inertial>
+  </link>
   <!-- ==================== Transmissions ==================== -->
   <transmission name="trans_base_rotation">

Commit message: feat: 添加眼在手上的摄像头 URDF/SRDF 定义和驱动 launch
URDF (dofbot.xacro):
- wrist_roll_link 下新增 camera_link (fixed joint)
- 安装位置 (0, 0.05, -0.05) 与 MJCF 中 camera 元素一致
- 无视觉几何体（已嵌入 wrist_roll_link 的 STL）
- 轻量惯量参数 (30g)

SRDF (dofbot.srdf):
- 新增 3 条 disable_collisions，排除 camera_link 与夹爪/腕部的自碰

Launch (camera.launch, 新建):
- usb_cam 节点, /dev/video0, YUYV 640x480
- 发布 /usb_cam/image_raw, frame_id=camera_link

硬件启动 (dofbot_hw.launch):
- include camera.launch

Co-Authored-By: Claude Opus 4.7 <noreply@anthropic.com>

File: dofbot_description/urdf/dofbot.xacro (robot description, xacro)
@@ -267,4 +267,18 @@
     </inertial>
   </link>
+  <!-- eye-in-hand camera, 安装位置与 MJCF 一致 (wrist_roll_link 下方) -->
+  <!-- 几何体已嵌入 wrist_roll_link 的 STL，此 link 仅用于 TF + 图像话题关联 -->
+  <joint name="camera_joint" type="fixed">
+    <origin xyz="0 0.05 -0.05" rpy="0 0 0"/>
+    <parent link="wrist_roll_link"/>
+    <child link="camera_link"/>
+  </joint>
+  <link name="camera_link">
+    <inertial>
+      <mass value="0.03"/>
+      <origin xyz="0 0 0"/>
+      <inertia ixx="1e-6" ixy="0" ixz="0" iyy="1e-6" iyz="0" izz="1e-6"/>
+    </inertial>
+  </link>
   <!-- ==================== Transmissions ==================== -->
   <transmission name="trans_base_rotation">
