Commit message: fix: ROS 最佳实践审计修复 — 构建依赖、参数化话题、异常处理

File: dofbot_description/urdf/deprecated/dofbot.urdf (robot description, URDF)
Before this commit: robot dofbot, 8 links, 7 joints
Links:
- link base_link: geometry collision mesh filename=package://dofbot_description/meshes/collision/base_link_col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; collision mesh filename=package://dofbot_description/meshes/collision/base_link_col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
- link link1: geometry collision mesh filename=package://dofbot_description/meshes/collision/link1_col.stl; visual mesh filename=package://dofbot_description/meshes/visual/link1.stl
- link link2: geometry collision mesh filename=package://dofbot_description/meshes/collision/link2_col_1.s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; collision mesh filename=package://dofbot_description/meshes/collision/link2_col_2.s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
- link link3: geometry collision mesh filename=package://dofbot_description/meshes/collision/link3_col_1.s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; collision mesh filename=package://dofbot_description/meshes/collision/link3_col_2.s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
- link link4: geometry collision mesh filename=package://dofbot_description/meshes/collision/link4_col_1.s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; collision mesh filename=package://dofbot_description/meshes/collision/link4_col_2.s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
